File: Adapter-CMRI8-RJ45.sch (EAGLE design)
At the start: 6 parts

Commit message: 2.0
Parts:
- added CON1: (no value), SPCoast:CONNECTOR-M08LOCK
Connections:
- removed net N$17: J1.1, J2.1, J3-1.S
- removed net N$18: J1.2, J2.2, J3-2.S
- removed net N$19: J1.3, J2.3, J3-3.S
- removed net N$2: JP1.1, JP2.1
- removed net N$20: J1.4, J2.4, J3-4.S
- removed net N$21: J1.5, J2.5, J3-5.S
- removed net N$22: J1.6, J2.6, J3-6.S
- removed net N$23: J1.7, J2.7, J3-7.S
- removed net N$24: J1.8, J2.8, J3-8.S
- removed net N$3: JP1.2, JP2.2
- new net GND: JP1.1, JP1.2, JP2.1, JP2.2
- new net L1: CON1.1, J1.1, J2.1, J3-1.S
- new net L2: CON1.2, J1.2, J2.2, J3-2.S
- new net L3: CON1.3, J1.3, J2.3, J3-3.S
- new net L4: CON1.4, J1.4, J2.4, J3-4.S
- new net L5: CON1.5, J1.5, J2.5, J3-5.S
- new net L6: CON1.6, J1.6, J2.6, J3-6.S
- new net L7: CON1.7, J1.7, J2.7, J3-7.S
- new net L8: CON1.8, J1.8, J2.8, J3-8.S
Other:
- note added: "v2.0"
- note removed: "v1.0"
- moved on the sheet: J2, J3-1, J3-2, J3-3, J3-4, J3-5, J3-6, J3-7, J3-8

Commit message: 3.0
Parts:
- removed JP1, JP2: (no value), SparkFun:M023.5MM_LOCK
- J1: value (none) -> RJ45; device con-amp:215877-7 -> SPCoast:CONNECTOR-RJ45-FRONT
- J2: device SparkFun:M083.5MM-8 -> SPCoast:CONNECTOR-M083.5MM-8
- J3: device con-molex:KK-156-8 -> SPCoast:KK-156-8F
Connections:
- removed net GND: JP1.1, JP1.2, JP2.1, JP2.2
Other:
- note removed: "Additional tie points"
Changed lines of the file:
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@@
 <?xml version="1.0" encoding="utf-8"?>
 <!DOCTYPE eagle SYSTEM "eagle.dtd">
-<eagle version="7.6.0">
+<eagle version="7.7.0">
 <drawing>
 <settings>
@@
 </classes>
 <parts>
-<part name="J1" library="con-amp" deviceset="215877-7" device=""/>
+<part name="J1" library="SPCoast" deviceset="CONNECTOR-RJ45" device="-FRONT" value="RJ45"/>
 <part name="FRAME1" library="SparkFun" deviceset="FRAME-LETTER" device=""/>
-<part name="J3" library="con-molex" deviceset="KK-156-8" device=""/>
-<part name="J2" library="SparkFun" deviceset="M08" device="3.5MM-8"/>
+<part name="J3" library="SPCoast" deviceset="KK-156-8" device="F"/>
+<part name="J2" library="SPCoast" deviceset="CONNECTOR-M08" device="3.5MM-8"/>
 <part name="U$1" library="SparkFun" deviceset="OSHW-LOGO" device="M"/>
-<part name="JP1" library="SparkFun" deviceset="M02" device="3.5MM_LOCK"/>
-<part name="JP2" library="SparkFun" deviceset="M02" device="3.5MM_LOCK"/>
 <part name="CON1" library="SPCoast" deviceset="CONNECTOR-M08" device="LOCK"/>
 </parts>
@@
 <text x="198.12" y="27.94" size="3.81" layer="104">RJ45 adapter</text>
 <text x="236.22" y="7.62" size="3.81" layer="104">v2.0</text>
-<text x="101.6" y="127" size="1.778" layer="94">Additional tie points</text>
 </plain>
 <instances>
-<instance part="J1" gate="G$1" x="134.62" y="93.98" rot="MR180"/>
+<instance part="J1" gate="J" x="134.62" y="93.98" rot="MR180"/>
 <instance part="FRAME1" gate="G$1" x="0" y="0"/>
 <instance part="FRAME1" gate="G$2" x="147.32" y="0"/>
@@
 <instance part="J2" gate="G$1" x="101.6" y="93.98"/>
 <instance part="U$1" gate="G$1" x="17.78" y="12.7"/>
-<instance part="JP1" gate="G$1" x="116.84" y="116.84"/>
-<instance part="JP2" gate="G$1" x="106.68" y="116.84"/>
 <instance part="CON1" gate="G$1" x="124.46" y="93.98"/>
 </instances>
@@
 <net name="L1" class="0">
 <segment>
-<wire x1="147.32" y1="86.36" x2="129.54" y2="86.36" width="0.1524" layer="91"/>
-<junction x="129.54" y="86.36"/>
-<pinref part="J1" gate="G$1" pin="1"/>
+<wire x1="147.32" y1="86.36" x2="132.08" y2="86.36" width="0.1524" layer="91"/>
+<junction x="132.08" y="86.36"/>
+<pinref part="J1" gate="J" pin="1"/>
 <pinref part="J3" gate="-1" pin="S"/>
 <pinref part="J2" gate="G$1" pin="1"/>
 <pinref part="CON1" gate="G$1" pin="1"/>
-<wire x1="129.54" y1="86.36" x2="106.68" y2="86.36" width="0.1524" layer="91"/>
+<wire x1="132.08" y1="86.36" x2="106.68" y2="86.36" width="0.1524" layer="91"/>
+<wire x1="129.54" y1="86.36" x2="132.08" y2="86.36" width="0.1524" layer="91"/>
 </segment>
 </net>
 <net name="L2" class="0">
 <segment>
-<wire x1="147.32" y1="88.9" x2="129.54" y2="88.9" width="0.1524" layer="91"/>
-<junction x="129.54" y="88.9"/>
-<pinref part="J1" gate="G$1" pin="2"/>
+<wire x1="147.32" y1="88.9" x2="132.08" y2="88.9" width="0.1524" layer="91"/>
+<junction x="132.08" y="88.9"/>
+<pinref part="J1" gate="J" pin="2"/>
 <pinref part="J3" gate="-2" pin="S"/>
 <pinref part="J2" gate="G$1" pin="2"/>
 <pinref part="CON1" gate="G$1" pin="2"/>
-<wire x1="129.54" y1="88.9" x2="106.68" y2="88.9" width="0.1524" layer="91"/>
+<wire x1="132.08" y1="88.9" x2="106.68" y2="88.9" width="0.1524" layer="91"/>
+<wire x1="129.54" y1="88.9" x2="132.08" y2="88.9" width="0.1524" layer="91"/>
 </segment>
 </net>
 <net name="L3" class="0">
 <segment>
-<wire x1="147.32" y1="91.44" x2="129.54" y2="91.44" width="0.1524" layer="91"/>
-<junction x="129.54" y="91.44"/>
-<pinref part="J1" gate="G$1" pin="3"/>
+<wire x1="147.32" y1="91.44" x2="132.08" y2="91.44" width="0.1524" layer="91"/>
+<junction x="132.08" y="91.44"/>
+<pinref part="J1" gate="J" pin="3"/>
 <pinref part="J3" gate="-3" pin="S"/>
 <pinref part="J2" gate="G$1" pin="3"/>
 <pinref part="CON1" gate="G$1" pin="3"/>
-<wire x1="129.54" y1="91.44" x2="106.68" y2="91.44" width="0.1524" layer="91"/>
+<wire x1="132.08" y1="91.44" x2="106.68" y2="91.44" width="0.1524" layer="91"/>
+<wire x1="129.54" y1="91.44" x2="132.08" y2="91.44" width="0.1524" layer="91"/>
 </segment>
 </net>
 <net name="L4" class="0">
 <segment>
-<wire x1="147.32" y1="93.98" x2="129.54" y2="93.98" width="0.1524" layer="91"/>
-<junction x="129.54" y="93.98"/>
-<pinref part="J1" gate="G$1" pin="4"/>
+<wire x1="147.32" y1="93.98" x2="132.08" y2="93.98" width="0.1524" layer="91"/>
+<junction x="132.08" y="93.98"/>
+<pinref part="J1" gate="J" pin="4"/>
 <pinref part="J3" gate="-4" pin="S"/>
 <pinref part="J2" gate="G$1" pin="4"/>
 <pinref part="CON1" gate="G$1" pin="4"/>
-<wire x1="129.54" y1="93.98" x2="106.68" y2="93.98" width="0.1524" layer="91"/>
+<wire x1="132.08" y1="93.98" x2="106.68" y2="93.98" width="0.1524" layer="91"/>
+<wire x1="129.54" y1="93.98" x2="132.08" y2="93.98" width="0.1524" layer="91"/>
 </segment>
 </net>
 <net name="L5" class="0">
 <segment>
-<wire x1="147.32" y1="96.52" x2="129.54" y2="96.52" width="0.1524" layer="91"/>
-<junction x="129.54" y="96.52"/>
-<pinref part="J1" gate="G$1" pin="5"/>
+<wire x1="147.32" y1="96.52" x2="132.08" y2="96.52" width="0.1524" layer="91"/>
+<junction x="132.08" y="96.52"/>
+<pinref part="J1" gate="J" pin="5"/>
 <pinref part="J3" gate="-5" pin="S"/>
 <pinref part="J2" gate="G$1" pin="5"/>
 <pinref part="CON1" gate="G$1" pin="5"/>
-<wire x1="129.54" y1="96.52" x2="106.68" y2="96.52" width="0.1524" layer="91"/>
+<wire x1="132.08" y1="96.52" x2="106.68" y2="96.52" width="0.1524" layer="91"/>
+<wire x1="129.54" y1="96.52" x2="132.08" y2="96.52" width="0.1524" layer="91"/>
 </segment>
 </net>
 <net name="L6" class="0">
 <segment>
-<wire x1="147.32" y1="99.06" x2="129.54" y2="99.06" width="0.1524" layer="91"/>
-<junction x="129.54" y="99.06"/>
-<pinref part="J1" gate="G$1" pin="6"/>
+<wire x1="147.32" y1="99.06" x2="132.08" y2="99.06" width="0.1524" layer="91"/>
+<junction x="132.08" y="99.06"/>
+<pinref part="J1" gate="J" pin="6"/>
 <pinref part="J3" gate="-6" pin="S"/>
 <pinref part="J2" gate="G$1" pin="6"/>
 <pinref part="CON1" gate="G$1" pin="6"/>
-<wire x1="129.54" y1="99.06" x2="106.68" y2="99.06" width="0.1524" layer="91"/>
+<wire x1="132.08" y1="99.06" x2="106.68" y2="99.06" width="0.1524" layer="91"/>
+<wire x1="129.54" y1="99.06" x2="132.08" y2="99.06" width="0.1524" layer="91"/>
 </segment>
 </net>
 <net name="L7" class="0">
 <segment>
-<wire x1="147.32" y1="101.6" x2="129.54" y2="101.6" width="0.1524" layer="91"/>
-<junction x="129.54" y="101.6"/>
-<pinref part="J1" gate="G$1" pin="7"/>
+<wire x1="147.32" y1="101.6" x2="132.08" y2="101.6" width="0.1524" layer="91"/>
+<junction x="132.08" y="101.6"/>
+<pinref part="J1" gate="J" pin="7"/>
 <pinref part="J3" gate="-7" pin="S"/>
 <pinref part="J2" gate="G$1" pin="7"/>
 <pinref part="CON1" gate="G$1" pin="7"/>
-<wire x1="129.54" y1="101.6" x2="106.68" y2="101.6" width="0.1524" layer="91"/>
+<wire x1="132.08" y1="101.6" x2="106.68" y2="101.6" width="0.1524" layer="91"/>
+<wire x1="129.54" y1="101.6" x2="132.08" y2="101.6" width="0.1524" layer="91"/>
 </segment>
 </net>
 <net name="L8" class="0">
 <segment>
-<wire x1="147.32" y1="104.14" x2="129.54" y2="104.14" width="0.1524" layer="91"/>
-<junction x="129.54" y="104.14"/>
-<pinref part="J1" gate="G$1" pin="8"/>
+<wire x1="147.32" y1="104.14" x2="132.08" y2="104.14" width="0.1524" layer="91"/>
+<junction x="132.08" y="104.14"/>
+<pinref part="J1" gate="J" pin="8"/>
 <pinref part="J3" gate="-8" pin="S"/>
 <pinref part="J2" gate="G$1" pin="8"/>
 <pinref part="CON1" gate="G$1" pin="8"/>
-<wire x1="129.54" y1="104.14" x2="106.68" y2="104.14" width="0.1524" layer="91"/>
-</segment>
-</net>
-<net name="GND" class="0">
-<segment>
-<wire x1="114.3" y1="119.38" x2="124.46" y2="119.38" width="0.1524" layer="91"/>
-<pinref part="JP1" gate="G$1" pin="2"/>
-<pinref part="JP2" gate="G$1" pin="2"/>
-<wire x1="114.3" y1="116.84" x2="124.46" y2="116.84" width="0.1524" layer="91"/>
-<pinref part="JP1" gate="G$1" pin="1"/>
-<pinref part="JP2" gate="G$1" pin="1"/>
-<wire x1="124.46" y1="119.38" x2="124.46" y2="116.84" width="0.1524" layer="91"/>
-<junction x="124.46" y="119.38"/>
-<junction x="124.46" y="116.84"/>
-</segment>
-</net>
+<wire x1="132.08" y1="104.14" x2="106.68" y2="104.14" width="0.1524" layer="91"/>
+<wire x1="129.54" y1="104.14" x2="132.08" y2="104.14" width="0.1524" layer="91"/>
+</segment>
+</net>

Commit message: 4.0
Parts:
- added J4: (no value), SPCoast:CONNECTOR-M04SCREW_LOCK
- added M1, M2: MOUNTINGHOLE, SPCoast:MOUNTINGHOLE
- added R1, R2, R3, R4, R5, R6, R7, R8: (no value), SPCoast:RPTH04
- U$1: value OSHW-LOGOM -> DOC-OSHW-LOGO-M; device SparkFun:OSHW-LOGOM -> SPCoast:DOC-OSHW-LOGO-M
- renumbered CON1 to J5
Connections:
- new net GND: J4.1, J4.2, J4.3, J4.4
- net L1: now also R1.1, R1.2
- net L2: now also R2.1, R2.2
- net L3: now also R3.1, R3.2
- net L4: now also R4.1, R4.2
- net L5: now also R5.1, R5.2
- net L6: now also R6.1, R6.2
- net L7: now also R7.1, R7.2
- net L8: now also R8.1, R8.2
Other:
- note added: "Ground tie points"
- note added: "v4.0"
- note removed: "v2.0"
- moved on the sheet: J1

Commit message: Addrd SPDT frog power connector
Parts:
- added CON1: CONNECTOR-M033.5MM-LOCK, SPCoast:CONNECTOR-M033.5MM-LOCK
- U$1: value DOC-OSHW-LOGO-M -> DOC-OSHW-LOGO-L; device SPCoast:DOC-OSHW-LOGO-M -> SPCoast:DOC-OSHW-LOGO-L
Connections:
- net L5: now also CON1.1
- net L6: now also CON1.2
- net L7: now also CON1.3
Other:
- note added: "3.5mm/3 Frog Power SPDT"
- note added: "V5.0 - Added Frog Power breakout"
- note added: "v5.0"
- note removed: "v4.0"
Changed lines of the file:
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@@
 <part name="J3" library="SPCoast" deviceset="KK-156-8" device="F"/>
 <part name="J2" library="SPCoast" deviceset="CONNECTOR-M08" device="3.5MM-8"/>
-<part name="U$1" library="SPCoast" deviceset="DOC-OSHW-LOGO-" device="M" value="DOC-OSHW-LOGO-M"/>
+<part name="U$1" library="SPCoast" deviceset="DOC-OSHW-LOGO-" device="L" value="DOC-OSHW-LOGO-L"/>
 <part name="J1" library="SPCoast" deviceset="CONNECTOR-RJ45" device="-FRONT" value="RJ45"/>
 <part name="J4" library="SPCoast" deviceset="CONNECTOR-M04" device="SCREW_LOCK"/>
@@
 <part name="R7" library="SPCoast" deviceset="R*" device="PTH04"/>
 <part name="R8" library="SPCoast" deviceset="R*" device="PTH04"/>
+<part name="CON1" library="SPCoast" deviceset="CONNECTOR-M03" device="3.5MM-LOCK"/>
 </parts>
 <sheets>
@@
 <text x="152.4" y="27.94" size="3.81" layer="91">CMRI Breakout</text>
 <text x="198.12" y="27.94" size="3.81" layer="91">RJ45 adapter</text>
-<text x="236.22" y="7.62" size="3.81" layer="91">v4.0</text>
+<text x="236.22" y="7.62" size="3.81" layer="91">v5.0</text>
 <text x="96.52" y="22.86" size="1.778" layer="91" rot="R90">Ground tie points</text>
+<text x="149.86" y="38.1" size="1.778" layer="91">V5.0 - Added Frog Power breakout</text>
+<text x="96.52" y="132.08" size="1.778" layer="91">3.5mm/3  Frog Power SPDT</text>
 </plain>
 <instances>
@@
 <instance part="R7" gate="R" x="83.82" y="109.22"/>
 <instance part="R8" gate="R" x="83.82" y="114.3"/>
+<instance part="CON1" gate="G$1" x="100.33" y="121.92"/>
 </instances>
 <busses>
@@
 <pinref part="J2" gate="G$1" pin="5"/>
 <wire x1="147.32" y1="96.52" x2="129.54" y2="96.52" width="0.1524" layer="91"/>
-<wire x1="129.54" y1="96.52" x2="106.68" y2="96.52" width="0.1524" layer="91"/>
+<wire x1="129.54" y1="96.52" x2="109.22" y2="96.52" width="0.1524" layer="91"/>
+<wire x1="109.22" y1="96.52" x2="106.68" y2="96.52" width="0.1524" layer="91"/>
 <wire x1="88.9" y1="99.06" x2="106.68" y2="96.52" width="0.1524" layer="91"/>
 <junction x="106.68" y="96.52"/>
@@
 <junction x="78.74" y="99.06"/>
 <junction x="88.9" y="99.06"/>
+<pinref part="CON1" gate="G$1" pin="1"/>
+<wire x1="106.68" y1="119.38" x2="109.22" y2="119.38" width="0.1524" layer="91"/>
+<wire x1="109.22" y1="119.38" x2="109.22" y2="96.52" width="0.1524" layer="91"/>
+<junction x="109.22" y="96.52"/>
 </segment>
 </net>
@@
 <pinref part="J2" gate="G$1" pin="6"/>
 <wire x1="147.32" y1="99.06" x2="129.54" y2="99.06" width="0.1524" layer="91"/>
-<wire x1="129.54" y1="99.06" x2="106.68" y2="99.06" width="0.1524" layer="91"/>
+<wire x1="129.54" y1="99.06" x2="111.76" y2="99.06" width="0.1524" layer="91"/>
+<wire x1="111.76" y1="99.06" x2="106.68" y2="99.06" width="0.1524" layer="91"/>
 <wire x1="88.9" y1="104.14" x2="106.68" y2="99.06" width="0.1524" layer="91"/>
 <junction x="106.68" y="99.06"/>
@@
 <junction x="78.74" y="104.14"/>
 <junction x="88.9" y="104.14"/>
+<pinref part="CON1" gate="G$1" pin="2"/>
+<wire x1="106.68" y1="121.92" x2="111.76" y2="121.92" width="0.1524" layer="91"/>
+<wire x1="111.76" y1="121.92" x2="111.76" y2="99.06" width="0.1524" layer="91"/>
+<junction x="111.76" y="99.06"/>
 </segment>
 </net>
@@
 <pinref part="J2" gate="G$1" pin="7"/>
 <wire x1="147.32" y1="101.6" x2="129.54" y2="101.6" width="0.1524" layer="91"/>
-<wire x1="129.54" y1="101.6" x2="106.68" y2="101.6" width="0.1524" layer="91"/>
+<wire x1="129.54" y1="101.6" x2="114.3" y2="101.6" width="0.1524" layer="91"/>
+<wire x1="114.3" y1="101.6" x2="106.68" y2="101.6" width="0.1524" layer="91"/>
 <wire x1="88.9" y1="109.22" x2="106.68" y2="101.6" width="0.1524" layer="91"/>
 <junction x="106.68" y="101.6"/>
@@
 <junction x="78.74" y="109.22"/>
 <junction x="88.9" y="109.22"/>
-</segment>
-</net>
+<pinref part="CON1" gate="G$1" pin="3"/>
+<wire x1="106.68" y1="124.46" x2="114.3" y2="124.46" width="0.1524" layer="91"/>
+<wire x1="114.3" y1="124.46" x2="114.3" y2="101.6" width="0.1524" layer="91"/>
+<junction x="114.3" y="101.6"/>
+</segment>
+</net>
